File: projects/8bitmixtape_nextleveledition_mixtape/current_version/working/working.kicad_sch (KiCad schematic)
At the start: 44 parts, among them Q1 BSS123, SW0 SWITCH_SMD, U5 ATMEGA32U41{colon}1, X1 USB_B_SMD, X2 PJ-327A, Y2 8MHz

Commit message: all brought together
Parts:
- removed BAT+0, BAT-0: SMD5, working:SMD2,54-5,08, symbol working-eagle-import:SMD5
- removed C11, C2, C3, C6, C8: 1uF, working:0603-CAP, symbol working-eagle-import:CAP0603-CAP
- removed C4: 0.1uF, working:0603-CAP, symbol working-eagle-import:CAP0603-CAP
- removed C5, C7: 22pF, working:0603-CAP, symbol working-eagle-import:CAP0603-CAP
- removed JP4: AVR_SPI_PRG_6PTH, working:2X3, symbol working-eagle-import:AVR_SPI_PRG_6PTH
- removed LED2: Blue, working:LED-0603, symbol working-eagle-import:LED0603
- removed LED4: Red, working:LED-0603, symbol working-eagle-import:LED0603
- removed LED5: Yellow, working:LED-0603, symbol working-eagle-import:LED0603
- removed LOGO1: OSHW-LOGOL, working:OSHW-LOGO-L, symbol working-eagle-import:OSHW-LOGOL
- removed PAD1, PAD2, PAD3: WIREPADSMD1,27-254, working:SMD1,27-2,54, symbol working-eagle-import:WIREPADSMD1,27-254
- removed POT_LEFT0, POT_RIGHT0: EVUA, working:EVUF, symbol working-eagle-import:EVUA
- removed Q1: BSS123, working:SOT23, symbol working-eagle-import:BSS123
- removed R1, R2: 33, working:0603-RES, symbol working-eagle-import:RESISTOR0603-RES
- removed R10, R16, R3, R4, R7: 330, working:0603-RES, symbol working-eagle-import:RESISTOR0603-RES
- removed R11, R12: 22, working:0603-RES, symbol working-eagle-import:RESISTOR0603-RES
- removed R14, R15: 10k, working:0603-RES, symbol working-eagle-import:RESISTOR0603-RES
- removed R6: 10K, working:0603-RES, symbol working-eagle-import:RESISTOR0603-RES
- removed S1: Left, working:TASTER-9314_SMD, symbol working-eagle-import:TASTER-9314_SMD
- removed S3: Right, working:TASTER-9314_SMD, symbol working-eagle-import:TASTER-9314_SMD
- removed SD0: MICROSD, working:MICROSD, symbol working-eagle-import:MICROSD
- removed SPEAKER0: PS603SPK, working:PS603, symbol working-eagle-import:PS603SPK
- removed SW0: SWITCH_SMD, working:SWITCH_SMD, symbol working-eagle-import:SWITCH_SMD
- removed U$1, U$2: FIDUCIAL, working:FIDUCIAL_1MM, symbol working-eagle-import:FIDUCIAL
- removed U5: ATMEGA32U41{colon}1, working:QFN-44-NOPAD_1_1, symbol working-eagle-import:ATMEGA32U41{colon}1
- removed X1: USB_B_SMD, working:USB_B_SMD, symbol working-eagle-import:USB_B_SMD
- removed X2: PJ-327A, working:PJ-327A, symbol working-eagle-import:PJ-327A
- removed Y2: 8MHz, working:CRYSTAL-SMD-5X3, symbol working-eagle-import:CRYSTAL5X3
Other:
- added sheet working_1 (working_1.kicad_sch)
- added sheet working_2 (working_2.kicad_sch)
- note removed: "Add Charge Status to ATmega"
- note removed: "Add battery voltage detect"
- note removed: "Change to 8MHz Xtal"
- note removed: "Change to ATmega32U4"
- note removed: "Changed PWM pin designator to ~"
- note removed: "Changed VCC to 3.3V"
- note removed: "Leah Buechley"
- note removed: "N. Seidle"
- note removed: "New on v31:"
- note removed: "New on v3:"
- note removed: "Re-arranged and re-named SPI pins"
- note removed: "Re-ordered Analog pins"
- note removed: "Removed FTDI Connection"
- note removed: "Shigeru Kobayashi"
- note removed: "Switch to microUSB"
- note removed: "T. Klopfenstein"
- note removed: "Update reset switch"
- note removed: "v31"
