File: projects/contextualelectronics_ce_soldering_practice_cesp/current_version/working/working.kicad_sch (KiCad schematic)
At the start: 5 parts

Commit message: working on gens
Parts:
- removed U?: LTC1594CS, TSSOP14, symbol CESP-rescue:LTC1594CS
- removed U?: TL074, TSSOP14, symbol CESP-rescue:TL074
- removed U? (x3): TL074, symbol CESP-rescue:TL074
- added U1: CE_HEADER, symbol ce_header:CE_HEADER
Other:
- note removed: "NOTE: THIS IS JUST A TEST BOARD REMOVE ALL COMPONENTS AND CREATE YOUR OWN INCLUDE SCHEMATIC HOOKUPS/NETLIST"
Changed lines of the file:
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@@
 (kicad_sch (version 20230121) (generator eeschema)
   (paper "A4")
-  (title_block
-    (date "24 jan 2014")
-  )
-  (text "NOTE: THIS IS JUST A TEST BOARD\nREMOVE ALL COMPONENTS AND CREATE YOUR OWN\nINCLUDE SCHEMATIC HOOKUPS/NETLIST"
-    (at 113.03 118.11 0)
-    (effects (font (size 2.032 2.032)) (justify left bottom))
-  )
-  (symbol (lib_id "CESP-rescue:LTC1594CS") (at 95.25 83.82 0) (unit 1)
+  (symbol (lib_id "ce_header:CE_HEADER") (at 92.71 82.55 0) (mirror x) (unit 1)
     (in_bom yes) (on_board yes) (dnp no)
-    (property "Reference" "U?" (at 95.25 67.31 0)
+    (property "Reference" "U1" (at 92.71 82.55 0)
       (effects (font (size 1.524 1.524)))
     )
-    (property "Value" "LTC1594CS" (at 95.25 100.33 0)
+    (property "Value" "CE_HEADER" (at 92.71 114.3 0)
       (effects (font (size 1.524 1.524)))
     )
-    (property "Footprint" "TSSOP14" (at 95.25 83.82 0)
-      (effects (font (size 1.524 1.524)))
+    (property "Footprint" "" (at 92.71 82.55 0)
+      (effects (font (size 1.524 1.524)) hide)
     )
-    (property "Datasheet" "" (at 95.25 83.82 0)
-      (effects (font (size 1.524 1.524)))
+    (property "Datasheet" "" (at 92.71 82.55 0)
+      (effects (font (size 1.524 1.524)) hide)
     )
     (pin "1")
     (pin "10")
-    (pin "11")
     (pin "12")
     (pin "13")
@@
     (pin "15")
     (pin "16")
-    (pin "2")
+    (pin "17")
+    (pin "18")
+    (pin "19")
     (pin "3")
     (pin "4")
@@
     (pin "7")
     (pin "8")
-    (pin "9")
     (instances
-      (project "CESP"
-        (path "/08f864b0-7135-4c7d-bb4a-f0789e917f2a"
-          (reference "U?") (unit 1)
+      (project "working"
+        (path "/61ea1fd5-9e28-4249-8f14-98e6efe1b589"
+          (reference "U1") (unit 1)
         )
       )
-    )
-  )
-  (symbol (lib_id "CESP-rescue:TL074") (at 181.61 54.61 0) (unit 1)
-    (in_bom yes) (on_board yes) (dnp no)
-    (property "Reference" "U?" (at 182.88 49.53 0)
-      (effects (font (size 1.524 1.524)))
-    )
-    (property "Value" "TL074" (at 185.42 59.69 0)
-      (effects (font (size 1.27 1.27)))
-    )
-    (property "Footprint" "TSSOP14" (at 181.61 54.61 0)
-      (effects (font (size 1.524 1.524)))
-    )
-    (property "Datasheet" "" (at 181.61 54.61 0)
-      (effects (font (size 1.524 1.524)))
-    )
-    (pin "11")
-    (pin "4")
-    (pin "1")
-    (pin "2")
-    (pin "3")
-    (pin "5")
-    (pin "6")
-    (pin "7")
-    (pin "10")
-    (pin "8")
-    (pin "9")
-    (pin "12")
-    (pin "13")
-    (pin "14")
-    (instances
-      (project "CESP"
-        (path "/08f864b0-7135-4c7d-bb4a-f0789e917f2a"
-          (reference "U?") (unit 1)
-        )
-      )
-    )
-  )
-  (symbol (lib_id "CESP-rescue:TL074") (at 182.88 88.9 0) (unit 2)
-    (in_bom yes) (on_board yes) (dnp no)
-    (property "Reference" "U?" (at 184.15 83.82 0)
-      (effects (font (size 1.524 1.524)))
-    )
-    (property "Value" "TL074" (at 186.69 93.98 0)
-      (effects (font (size 1.27 1.27)))
-    )
-    (property "Footprint" "" (at 182.88 88.9 0)
-      (effects (font (size 1.524 1.524)))
-    )
-    (property "Datasheet" "" (at 182.88 88.9 0)
-      (effects (font (size 1.524 1.524)))
-    )
-    (pin "11")
-    (pin "4")
-    (pin "1")
-    (pin "2")
-    (pin "3")
-    (pin "5")
-    (pin "6")
-    (pin "7")
-    (pin "10")
-    (pin "8")
-    (pin "9")
-    (pin "12")
-    (pin "13")
-    (pin "14")
-    (instances
-      (project "CESP"
-        (path "/08f864b0-7135-4c7d-bb4a-f0789e917f2a"
-          (reference "U?") (unit 2)
-        )
-      )
-    )
-  )
-  (symbol (lib_id "CESP-rescue:TL074") (at 218.44 88.9 0) (unit 1)
-    (in_bom yes) (on_board yes) (dnp no)
-    (property "Reference" "U?" (at 219.71 83.82 0)
-      (effects (font (size 1.524 1.524)))
-    )
-    (property "Value" "TL074" (at 222.25 93.98 0)
-      (effects (font (size 1.27 1.27)))
-    )
-    (property "Footprint" "" (at 218.44 88.9 0)
-      (effects (font (size 1.524 1.524)))
-    )
-    (property "Datasheet" "" (at 218.44 88.9 0)
-      (effects (font (size 1.524 1.524)))
-    )
-    (pin "11")
-    (pin "4")
-    (pin "1")
-    (pin "2")
-    (pin "3")
-    (pin "5")
-    (pin "6")
-    (pin "7")
-    (pin "10")
-    (pin "8")
-    (pin "9")
-    (pin "12")
-    (pin "13")
-    (pin "14")
-    (instances
-      (project "CESP"
-        (path "/08f864b0-7135-4c7d-bb4a-f0789e917f2a"
-          (reference "U?") (unit 1)
-        )
-      )
-    )
-  )
-  (symbol (lib_id "CESP-rescue:TL074") (at 217.17 53.34 0) (unit 1)
-    (in_bom yes) (on_board yes) (dnp no)
-    (property "Reference" "U?" (at 218.44 48.26 0)
-      (effects (font (size 1.524 1.524)))
-    )
-    (property "Value" "TL074" (at 220.98 58.42 0)
-      (effects (font (size 1.27 1.27)))
-    )
-    (property "Footprint" "" (at 217.17 53.34 0)
-      (effects (font (size 1.524 1.524)))
-    )
-    (property "Datasheet" "" (at 217.17 53.34 0)
-      (effects (font (size 1.524 1.524)))
-    )
-    (pin "11")
-    (pin "4")
-    (pin "1")
-    (pin "2")
-    (pin "3")
-    (pin "5")
-    (pin "6")
-    (pin "7")
-    (pin "10")
-    (pin "8")
-    (pin "9")
-    (pin "12")
-    (pin "13")
-    (pin "14")
-    (instances
-      (project "CESP"
-        (path "/08f864b0-7135-4c7d-bb4a-f0789e917f2a"
-          (reference "U?") (unit 1)
-        )
-      )
